File: PCB/FELLeveler/FELLeveler.kicad_pcb (KiCad board)
At the start: 2 copper layers, 16 parts, among them J1 PRG0, J2 PRG1, T1 VCC IN, U1 ESP32-WROOM-32

Commit message: Initial positioning
Parts:
- added REF**: MountingHole_2.5mm, MountingHole:MountingHole_2.5mm, F.Cu at (164.0, 127.0)
- H1, H2, H3: moved to B.Cu
- moved H1 45.1 mm to (134.2, 113.1), turned to 0 degrees
- moved T1 40.8 mm to (135.0, 120.0), turned to -90 degrees
- moved H4 31.5 mm to (162.8, 118.8)
- moved J2 29.9 mm to (162.8, 100.5)
- moved C2 27.0 mm to (139.4, 95.5)
- moved C3 27.0 mm to (139.4, 100.5)
- moved R1 27.0 mm to (137.1, 100.5)
- moved U1 27.0 mm to (150.7, 102.5)
- moved C1 27.0 mm to (136.7, 96.1)
- moved H2 25.6 mm to (159.0, 115.6), turned to 90 degrees
- moved J1 24.3 mm to (166.5, 103.0)
- moved REF** 20.2 mm to (136.5, 127.0)
- moved L1 17.2 mm to (168.0, 122.3), turned to -90 degrees
- moved H3 17.2 mm to (143.8, 115.6), turned to 90 degrees
- moved R7 12.4 mm to (167.0, 119.0)
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Routing:
- net /STATUS_LED: track 1.16 -> 0.00 mm
- net unconnected-(U1-Pad27): track 0.99 -> 0.00 mm, vias 1 -> 0
- net unconnected-(U1-Pad26): vias 1 -> 0
Other:
- board outline added: 37 x 37 mm
- board text added: "GND"
- board text added: "SDA"
- board text added: "VCC"
- board text added: "VDD"

Commit message: PCB routed
Parts:
- moved REF** 0.50 mm to (163.5, 127.0)
Routing:
- net VDD: track 27.6 -> 81.5 mm
- net /SCL: track 0.00 -> 33.9 mm
- net /SDA: track 0.00 -> 29.8 mm
- net /IO12: track 0.00 -> 27.4 mm, vias 0 -> 2
- net /DIN: track 0.00 -> 22.6 mm, vias 0 -> 1
- net /IO0: track 0.38 -> 18.1 mm
- net /STATUS_LED: track 0.00 -> 13.5 mm, vias 0 -> 2
- net /EN: track 19.8 -> 30.5 mm
- net /TXD0: track 0.00 -> 10.2 mm, vias 0 -> 1
- net /CLK: track 0.00 -> 8.96 mm, vias 0 -> 1
- net VCC: track 0.00 -> 8.77 mm
- net /RXD0: track 0.00 -> 7.93 mm, vias 0 -> 1
- net /CS: track 0.00 -> 4.86 mm, vias 0 -> 1
- net /DC: track 0.90 -> 3.92 mm
- net Net-(L1-Pad1): track 0.00 -> 2.41 mm
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- added copper zone on B.Cu, net GND
- added copper zone on F.Cu, net GND

Commit message: Added Boot pin, tweaked PCB
Parts:
- added JP1: Boot Jumper, Jumper:SolderJumper-2_P1.3mm_Bridged_Pad1.0x1.5mm, B.Cu at (146.7, 107.5)
- moved H1 5.35 mm to (139.5, 112.0)
Connections:
- U1 pad 13: unconnected-(U1-Pad13) -> /BOOT
Routing:
- net /BOOT: track 0.00 -> 4.65 mm, vias 0 -> 1
- net VCC: track 8.77 -> 10.6 mm
- net VDD: track 81.5 -> 80.3 mm

Commit message: Tweaked PCB, submitted v1.0 to fab.
Parts:
- JP1: value Boot Jumper -> Boot; footprint Jumper:SolderJumper-2_P1.3mm_Bridged_Pad1.0x1.5mm -> Jumper:SolderJumper-2_P1.3mm_Open_Pad1.0x1.5mm; moved to F.Cu
- moved JP1 10.7 mm to (136.0, 107.7), turned to 90 degrees
- moved L1 4.75 mm to (168.0, 127.1)
Routing:
- net Net-(L1-Pad1): track 2.41 -> 7.16 mm
- net VDD: track 80.3 -> 84.6 mm
- net /BOOT: track 4.65 -> 6.62 mm, vias 1 -> 0
- net GND: vias 11 -> 14
Changed lines of the file:
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@@
       (effects (font (size 1 1) (thickness 0.15)))
+    )
+    (fp_text user "KEEP-OUT ZONE" (at 0 -19) (layer "Cmts.User")
+      (effects (font (size 1 1) (thickness 0.15)))
+    )
+    (fp_text user "5 mm" (at 7.8 -19.075 90) (layer "Cmts.User")
+      (effects (font (size 0.5 0.5) (thickness 0.1)))
     )
     (fp_text user "5 mm" (at 11.8 -14.375) (layer "Cmts.User")
       (effects (font (size 0.5 0.5) (thickness 0.1)))
-    )
-    (fp_text user "5 mm" (at 7.8 -19.075 90) (layer "Cmts.User")
-      (effects (font (size 0.5 0.5) (thickness 0.1)))
-    )
-    (fp_text user "KEEP-OUT ZONE" (at 0 -19) (layer "Cmts.User")
-      (effects (font (size 1 1) (thickness 0.15)))
     )
     (fp_text user "5 mm" (at -11.2 -14.375) (layer "Cmts.User")
@@
   )
   (footprint "LED_SMD:LED_0805_2012Metric" (layer "F.Cu")
-    (at 168 122.3125 -90)
+    (at 168 127.0625 -90)
     (descr "LED SMD 0805 (2012 Metric), square (rectangular) end terminal, IPC_7351 nominal, (Body size source: https://docs.google.com/spreadsheets/d/1BsfQQcO9C6DZCsRaXUlFlo91Tg2WpOkGARC1WS5S8t0/edit?usp=sharing), generated with kicad-footprint-generator")
     (tags "LED")
@@
       (rotate (xyz 0 0 0))
     )
+  )
+  (footprint "Jumper:SolderJumper-2_P1.3mm_Open_Pad1.0x1.5mm" (layer "F.Cu")
+    (at 136 107.65 90)
+    (descr "SMD Solder Jumper, 1x1.5mm Pads, 0.3mm gap, open")
+    (tags "solder jumper open")
+    (property "Sheetfile" "FELLeveler.kicad_sch")
+    (property "Sheetname" "")
+    (attr exclude_from_pos_files)
+    (fp_text reference "JP1" (at 0 -1.8 90) (layer "F.SilkS")
+      (effects (font (size 1 1) (thickness 0.15)))
+    )
+    (fp_text value "Boot" (at 0 1.9 90) (layer "F.Fab")
+      (effects (font (size 1 1) (thickness 0.15)))
+    )
+    (fp_line (start -1.4 -1) (end 1.4 -1) (layer "F.SilkS") (width 0.12))
+    (fp_line (start -1.4 1) (end -1.4 -1) (layer "F.SilkS") (width 0.12))
+    (fp_line (start 1.4 1) (end -1.4 1) (layer "F.SilkS") (width 0.12))
+    (fp_line (start 1.4 -1) (end 1.4 1) (layer "F.SilkS") (width 0.12))
+    (fp_line (start 1.65 1.25) (end 1.65 -1.25) (layer "F.CrtYd") (width 0.05))
+    (fp_line (start -1.65 -1.25) (end 1.65 -1.25) (layer "F.CrtYd") (width 0.05))
+    (fp_line (start -1.65 -1.25) (end -1.65 1.25) (layer "F.CrtYd") (width 0.05))
+    (fp_line (start 1.65 1.25) (end -1.65 1.25) (layer "F.CrtYd") (width 0.05))
+    (pad "1" smd rect (at -0.65 0 90) (size 1 1.5) (layers "F.Cu" "F.Mask")
+      (net 28 "/BOOT") (pinfunction "A") (pintype "passive"))
+    (pad "2" smd rect (at 0.65 0 90) (size 1 1.5) (layers "F.Cu" "F.Mask")
+      (net 1 "GND") (pinfunction "B") (pintype "passive"))
   )
   (footprint "Connector_PinHeader_2.54mm:PinHeader_1x04_P2.54mm_Vertical" (layer "F.Cu")
@@
     )
   )
-  (footprint "Jumper:SolderJumper-2_P1.3mm_Bridged_Pad1.0x1.5mm" (layer "B.Cu")
-    (at 146.65 107.5)
-    (descr "SMD Solder Jumper, 1x1.5mm Pads, 0.3mm gap, bridged with 1 copper strip")
-    (tags "net tie solder jumper bridged")
-    (property "Sheetfile" "FELLeveler.kicad_sch")
-    (property "Sheetname" "")
-    (attr exclude_from_pos_files)
-    (fp_text reference "JP1" (at 0 -2) (layer "B.SilkS")
-      (effects (font (size 1 1) (thickness 0.15)) (justify mirror))
-    )
-    (fp_text value "Boot Jumper" (at 0 -1.9) (layer "B.Fab")
-      (effects (font (size 1 1) (thickness 0.15)) (justify mirror))
-    )
-    (fp_poly (pts
-        (xy -0.25 0.3)
-        (xy 0.25 0.3)
-        (xy 0.25 -0.3)
-        (xy -0.25 -0.3)
-      ) (layer "B.Cu") (width 0) (fill solid))
-    (fp_line (start 1.4 1) (end 1.4 -1) (layer "B.SilkS") (width 0.12))
-    (fp_line (start 1.4 -1) (end -1.4 -1) (layer "B.SilkS") (width 0.12))
-    (fp_line (start -1.4 -1) (end -1.4 1) (layer "B.SilkS") (width 0.12))
-    (fp_line (start -1.4 1) (end 1.4 1) (layer "B.SilkS") (width 0.12))
-    (fp_line (start 1.65 -1.25) (end 1.65 1.25) (layer "B.CrtYd") (width 0.05))
-    (fp_line (start 1.65 -1.25) (end -1.65 -1.25) (layer "B.CrtYd") (width 0.05))
-    (fp_line (start -1.65 1.25) (end 1.65 1.25) (layer "B.CrtYd") (width 0.05))
-    (fp_line (start -1.65 1.25) (end -1.65 -1.25) (layer "B.CrtYd") (width 0.05))
-    (pad "1" smd rect (at -0.65 0) (size 1 1.5) (layers "B.Cu" "B.Mask")
-      (net 28 "/BOOT") (pinfunction "A") (pintype "passive"))
-    (pad "2" smd rect (at 0.65 0) (size 1 1.5) (layers "B.Cu" "B.Mask")
-      (net 1 "GND") (pinfunction "B") (pintype "passive"))
-  )
   (footprint "Connector_PinSocket_2.54mm:PinSocket_1x02_P2.54mm_Horizontal" (layer "B.Cu")
     (at 143.764 115.6 90)
@@
   (gr_rect (start 124.5 113.71) (end 144.5 102.71) (layer "Dwgs.User") (width 0.1) (fill none))
   (gr_rect (start 132.5 93) (end 169.5 130) (layer "Edge.Cuts") (width 0.05) (fill none))
-  (gr_text "FELLeveler\nv1.0" (at 149.9 127.9) (layer "F.SilkS")
-    (effects (font (size 1 1) (thickness 0.15)))
+  (gr_text "FELLeveler\nv1.0" (at 150 127) (layer "F.SilkS")
+    (effects (font (size 2 2) (thickness 0.3)))
   )
   (gr_text "SDA" (at 143.86 117.6) (layer "Dwgs.User")
@@
   (via (at 149.65 99.7) (size 0.6858) (drill 0.3302) (layers "F.Cu" "B.Cu") (net 1))
   (via (at 144.9 111.7) (size 0.6858) (drill 0.3302) (layers "F.Cu" "B.Cu") (net 1))
+  (via (at 163.5 103.5) (size 0.6858) (drill 0.3302) (layers "F.Cu" "B.Cu") (free) (net 1))
+  (via (at 160.5 113.5) (size 0.6858) (drill 0.3302) (layers "F.Cu" "B.Cu") (free) (net 1))
   (via (at 149.65 101.7) (size 0.6858) (drill 0.3302) (layers "F.Cu" "B.Cu") (net 1))
   (via (at 147.65 101.7) (size 0.6858) (drill 0.3302) (layers "F.Cu" "B.Cu") (net 1))
   (via (at 151.65 103.7) (size 0.6858) (drill 0.3302) (layers "F.Cu" "B.Cu") (net 1))
+  (via (at 162 103.5) (size 0.6858) (drill 0.3302) (layers "F.Cu" "B.Cu") (free) (net 1))
   (via (at 147.65 99.7) (size 0.6858) (drill 0.3302) (layers "F.Cu" "B.Cu") (net 1))
   (segment (start 135 114) (end 135 118.25) (width 0.4064) (layer "F.Cu") (net 2))
@@
   (segment (start 137.775 96.45) (end 136.65 97.575) (width 0.4572) (layer "F.Cu") (net 7))
   (segment (start 135.85 100.2125) (end 137.05 101.4125) (width 0.4572) (layer "F.Cu") (net 7))
+  (segment (start 166.5 122.575) (end 166.5 126.5) (width 0.4064) (layer "F.Cu") (net 7))
+  (segment (start 162.75 118.825) (end 166.5 122.575) (width 0.4064) (layer "F.Cu") (net 7))
   (segment (start 168 108.695) (end 167.65 109.045) (width 0.4572) (layer "F.Cu") (net 7))
   (segment (start 136.65 97.575) (end 135.85 98.375) (width 0.4572) (layer "F.Cu") (net 7))
   (segment (start 135.85 98.375) (end 135.85 100.2125) (width 0.4572) (layer "F.Cu") (net 7))
-  (segment (start 162.75 118.825) (end 163.575 118.825) (width 0.4064) (layer "F.Cu") (net 7))
   (segment (start 139.45 96.45) (end 140.43 95.47) (width 0.4572) (layer "F.Cu") (net 7))
   (segment (start 137.05 101.97) (end 137.05 101.4125) (width 0.4064) (layer "F.Cu") (net 7))
   (segment (start 143.85 95.5) (end 142.18 95.5) (width 0.4572) (layer "F.Cu") (net 7))
+  (segment (start 166.5 126.5) (end 168 128) (width 0.4064) (layer "F.Cu") (net 7))
   (segment (start 142.18 95.5) (end 142.15 95.47) (width 0.4572) (layer "F.Cu") (net 7))
-  (segment (start 163.575 118.825) (end 168 123.25) (width 0.4064) (layer "F.Cu") (net 7))
   (via (at 143.85 95.5) (size 0.6858) (drill 0.3302) (layers "F.Cu" "B.Cu") (net 7))
   (segment (start 160.6 95.5) (end 161.8 96.7) (width 0.4572) (layer "B.Cu") (net 7))
@@
   (segment (start 163.985 97.985) (end 164.6 98.6) (width 0.2032) (layer "F.Cu") (net 10))
   (segment (start 160.8 110.4) (end 160.49 110.71) (width 0.2032) (layer "F.Cu") (net 10))
-  (segment (start 167.9125 121.2875) (end 168 121.375) (width 0.2032) (layer "F.Cu") (net 11))
-  (segment (start 167.9125 119) (end 167.9125 121.2875) (width 0.2032) (layer "F.Cu") (net 11))
+  (segment (start 167.9125 119) (end 167.9125 126.0375) (width 0.2032) (layer "F.Cu") (net 11))
+  (segment (start 167.9125 126.0375) (end 168 126.125) (width 0.2032) (layer "F.Cu") (net 11))
   (via (at 159.15 104.36) (size 0.6858) (drill 0.3302) (layers "F.Cu" "B.Cu") (net 12))
   (segment (start 158.4 105.11) (end 159.15 104.36) (width 0.2032) (layer "B.Cu") (net 12))
@@
   (segment (start 142.15 110.85) (end 142.15 110.71) (width 0.2032) (layer "B.Cu") (net 15))
   (segment (start 144.7 113.4) (end 142.15 110.85) (width 0.2032) (layer "B.Cu") (net 15))
-  (via (at 142.15 109.44) (size 0.6858) (drill 0.3302) (layers "F.Cu" "B.Cu") (net 28))
-  (segment (start 143.56 109.44) (end 142.15 109.44) (width 0.2032) (layer "B.Cu") (net 28))
-  (segment (start 145.5 107.5) (end 143.56 109.44) (width 0.2032) (layer "B.Cu") (net 28))
-  (segment (start 146 107.5) (end 145.5 107.5) (width 0.2032) (layer "B.Cu") (net 28))
+  (segment (start 136 108.3) (end 140.3 108.3) (width 0.2032) (layer "F.Cu") (net 28))
+  (segment (start 140.3 108.3) (end 141.44 109.44) (width 0.2032) (layer "F.Cu") (net 28))
+  (segment (start 141.44 109.44) (end 142.15 109.44) (width 0.2032) (layer "F.Cu") (net 28))
   (segment (start 160.6 114.8) (end 159 113.2) (width 0.2032) (layer "F.Cu") (net 39))
   (segment (start 162 117.5) (end 160.6 116.1) (width 0.2032) (layer "F.Cu") (net 39))
